File: v2_plate_kicad/chocolatebarplate.kicad_pcb (KiCad board)
At the start: 2 copper layers, 313 x 100.3 mm, 0 parts

Commit message: v2
Parts:
- added G***: LOGO, platebacking:plateback, B.Cu at (139.2, 94.1)
Other:
- board size 313 x 100.3 mm -> 319 x 106.3 mm
