File: v2_kicad/chocolatebar.kicad_pcb (KiCad board)
At the start: 2 copper layers, 301.3 x 89.5 mm, 156 parts, among them J1 Conn_01x04, SW1 SW_Push, U1 ATmega32U4-AU, Y1 Crystal_GND24_Small

Commit message: v2
Parts:
- removed G***: LOGO, karin:chocobar

Commit message: V2 update
Parts:
- removed USB1: HRO-TYPE-C-31-M-12, Type-C:HRO-TYPE-C-31-M-12-HandSoldering
- added G***: LOGO, random-keyboard-parts:chocbar, B.Cu at (173.8, 53.2)
- added J2: USB_C_Receptacle_USB2.0, Modified Footprints:USB_C_Receptacle_HRO_TYPE-C-31-M-12, B.Cu at (40.0, 11.1)
Routing:
- added copper zone on B.Cu, net GND
- added copper zone on F.Cu, net GND
